Commit message: Added camera to URDF + improved readability

File: lbr_description/urdf/left_arm/left_arm.urdf.xacro (robot description, xacro)
@@ -48,203 +48,127 @@
   <joint name="table_to_pole" type="fixed">
     <parent link="table"/>
-    <child link="pole_link1"/>
+    <child link="base_link"/>
     <origin xyz="0 -0.35 0.015" rpy="0 0 0"/>
   </joint>
-  <link
-    name="pole_link1">
-    <inertial>
-      <origin
-        xyz="-2.0651E-17 0.006 -3.0598E-17"
-        rpy="0 0 0" />
-      <mass
-        value="0.67747" />
-      <inertia
-        ixx="0.0032039"
-        ixy="-2.5621E-20"
-        ixz="1.8363E-19"
-        iyy="0.0063916"
-        iyz="4.6661E-21"
-        izz="0.0032039" />
-    </inertial>
-    <visual>
-      <origin
-        xyz="0 0 0"
-        rpy="0 0 0" />
-      <geometry>
-        <mesh
-          filename="package://lbr_description/meshes/iiwa7/pole/pole_link1.STL" />
-      </geometry>
-      <material
-        name="">
-        <color
-          rgba="0.89412 0.91373 0.92941 1" />
-      </material>
-    </visual>
-    <collision>
-      <origin
-        xyz="0 0 0"
-        rpy="0 0 0" />
-      <geometry>
-        <mesh
-          filename="package://lbr_description/meshes/iiwa7/pole/pole_link1.STL" />
-      </geometry>
-    </collision>
-  </link>
-  <link
-    name="pole_link2">
-    <inertial>
-      <origin
-        xyz="0.08 0.004973 -0.08"
-        rpy="0 0 0" />
-      <mass
-        value="0.66701" />
-      <inertia
-        ixx="0.0014197"
-        ixy="-1.7809E-21"
-        ixz="-6.3093E-20"
-        iyy="0.0028283"
-        iyz="4.3854E-22"
-        izz="0.0014197" />
-    </inertial>
-    <visual>
-      <origin
-        xyz="0 0 0"
-        rpy="0 0 0" />
-      <geometry>
-        <mesh
-          filename="package://lbr_description/meshes/iiwa7/pole/pole_link2.STL" />
-      </geometry>
-      <material
-        name="">
-        <color
-          rgba="0.89804 0.91765 0.92941 1" />
-      </material>
-    </visual>
-    <collision>
-      <origin
-        xyz="0 0 0"
-        rpy="0 0 0" />
-      <geometry>
-        <mesh
-          filename="package://lbr_description/meshes/iiwa7/pole/pole_link2.STL" />
-      </geometry>
-    </collision>
-  </link>
-  <joint
-    name="pole_joint1"
-    type="fixed">
-    <origin
-      xyz="0.08 0.08 0.012"
-      rpy="1.5708 0 3.1416" />
-    <parent
-      link="pole_link1" />
-    <child
-      link="pole_link2" />
-    <axis
-      xyz="0 0 0" />
-  </joint>
-  <link
-    name="pole_link3">
-    <inertial>
-      <origin
-        xyz="-1.2525E-16 -0.7 -6.7084E-17"
-        rpy="0 0 0" />
-      <mass
-        value="2.7358" />
-      <inertia
-        ixx="0.083946"
-        ixy="-5.4209E-18"
-        ixz="3.7385E-19"
-        iyy="0.0037448"
-        iyz="-9.0633E-18"
-        izz="0.083945" />
-    </inertial>
-    <visual>
-      <origin
-        xyz="0 0 0"
-        rpy="0 0 0" />
-      <geometry>
-        <mesh
-          filename="package://lbr_description/meshes/iiwa7/pole/pole_link3.STL" />
-      </geometry>
-      <material
-        name="">
-        <color
-          rgba="0.89804 0.91765 0.92941 1" />
-      </material>
-    </visual>
-    <collision>
-      <origin
-        xyz="0 0 0"
-        rpy="0 0 0" />
-      <geometry>
-        <mesh
-          filename="package://lbr_description/meshes/iiwa7/pole/pole_link3.STL" />
-      </geometry>
-    </collision>
-  </link>
-  <joint
-    name="pole_joint2"
-    type="fixed">
-    <origin
-      xyz="0.08 1.01 -0.08"
-      rpy="0 0 0" />
-    <parent
-      link="pole_link2" />
-    <child
-      link="pole_link3" />
-    <axis
-      xyz="0 0 0" />
-  </joint>
-  <link
-    name="pole_link4">
-    <inertial>
-      <origin
-        xyz="-0.040013 -0.029602 -0.042411"
-        rpy="0 0 0" />
-      <mass
-        value="2.5894" />
-      <inertia
-        ixx="0.0034613"
-        ixy="-1.1553E-08"
-        ixz="-7.2089E-07"
-        iyy="0.031728"
-        iyz="-3.8836E-08"
-        izz="0.031631" />
-    </inertial>
-    <visual>
-      <origin
-        xyz="0 0 0"
-        rpy="0 0 0" />
-      <geometry>
-        <mesh
-          filename="package://lbr_description/meshes/iiwa7/pole/pole_link4.STL" />
-      </geometry>
-      <material
-        name="">
-        <color
-          rgba="0.89804 0.91765 0.92941 1" />
-      </material>
-    </visual>
-    <collision>
-      <origin
-        xyz="0 0 0"
-        rpy="0 0 0" />
-      <geometry>
-        <mesh
-          filename="package://lbr_description/meshes/iiwa7/pole/pole_link4.STL" />
-      </geometry>
-    </collision>
-  </link>
-  <joint
-    name="pole_joint3"
-    type="fixed">
-    <origin
-      xyz="0.04 -0.76 0.04"
-      rpy="-1.5708 0 0" />
-    <parent
-      link="pole_link3" />
-    <child
-      link="pole_link4" />
+ <link
+    name="base_link">
+    <inertial>
+      <origin
+        xyz="-4.60531013034323E-05 0.0269896752933545 0.220110783524606"
+        rpy="0 0 0" />
+      <mass
+        value="6.67768952534525" />
+      <inertia
+        ixx="0.0927060188022499"
+        ixy="-1.15527252193294E-08"
+        ixz="9.95970442619751E-05"
+        iyy="0.120986260169313"
+        iyz="3.8835854033819E-08"
+        izz="0.0446111571845848" />
+    </inertial>
+    <visual>
+      <origin
+        xyz="0 0 0"
+        rpy="0 0 0" />
+      <geometry>
+        <mesh
+          filename="package://lbr_description/meshes/pole/base_link.STL" />
+      </geometry>
+      <material
+        name="">
+        <color
+          rgba="0.894117647058823 0.913725490196078 0.929411764705882 1" />
+      </material>
+    </visual>
+    <collision>
+      <origin
+        xyz="0 0 0"
+        rpy="0 0 0" />
+      <geometry>
+        <mesh
+          filename="package://lbr_description/meshes/pole/base_link.STL" />
+      </geometry>
+    </collision>
+  </link>
+  <link
+    name="camera_mount">
+    <inertial>
+      <origin
+        xyz="-0.00320794759811641 -0.045 -0.0149674652046672"
+        rpy="0 0 0" />
+      <mass
+        value="0.26247066782014" />
+      <inertia
+        ixx="0.000291627708890385"
+        ixy="-1.26470935677167E-20"
+        ixz="-2.87105610515067E-05"
+        iyy="0.0003118294834033"
+        iyz="1.66734346017947E-20"
+        izz="0.000247269374096239" />
+    </inertial>
+    <visual>
+      <origin
+        xyz="0 0 0"
+        rpy="0 0 0" />
+      <geometry>
+        <mesh
+          filename="package://lbr_description/meshes/pole/camera_mount.STL" />
+      </geometry>
+      <material
+        name="">
+        <color
+          rgba="0.792156862745098 0.819607843137255 0.933333333333333 1" />
+      </material>
+    </visual>
+    <collision>
+      <origin
+        xyz="0 0 0"
+        rpy="0 0 0" />
+      <geometry>
+        <mesh
+          filename="package://lbr_description/meshes/pole/camera_mount.STL" />
+      </geometry>
+    </collision>
+  </link>
+  <joint
+    name="base_to_camera_mount"
+    type="fixed">
+    <origin
+      xyz="-0.045 0 0.6319"
+      rpy="3.14159265358979 0 -1.5707963267949" />
+    <parent
+      link="base_link" />
+    <child
+      link="camera_mount" />
+    <axis
+      xyz="0 0 0" />
+  </joint>
+  <link
+    name="camera_base">
+    <inertial>
+      <origin
+        xyz="0.00152788225160483 -3.4246869961186E-07 0.0122350480077058"
+        rpy="0 0 0" />
+      <mass
+        value="0.0481481386626754" />
+      <inertia
+        ixx="2.73639159474837E-05"
+        ixy="-4.26051115035423E-07"
+        ixz="7.54720864413178E-09"
+        iyy="3.35044769883872E-06"
+        iyz="2.12843084673675E-09"
+        izz="2.66245899513959E-05" />
+    </inertial>
+  </link>
+  <joint
+    name="camera_mount_to_camera"
+    type="fixed">
+    <origin
+      xyz="-0.0615 -0.045 -0.0545999999999999"
+      rpy="-3.14159265358979 -0.97738438111683 3.14159265358979" />
+    <parent
+      link="camera_mount" />
+    <child
+      link="camera_base" />
     <axis
       xyz="0 0 0" />
@@ -254,48 +178,48 @@
     <inertial>
       <origin
-        xyz="1.0186E-07 0.0021716 0.018156"
-        rpy="0 0 0" />
-      <mass
-        value="0.38712" />
-      <inertia
-        ixx="0.00048365"
-        ixy="8.1163E-10"
-        ixz="8.7467E-10"
-        iyy="0.00098031"
-        iyz="-1.8644E-05"
-        izz="0.0012915" />
-    </inertial>
-    <visual>
-      <origin
-        xyz="0 0 0"
-        rpy="0 0 0" />
-      <geometry>
-        <mesh
-          filename="package://lbr_description/meshes/iiwa7/pole/pole_link5_1.STL" />
-      </geometry>
-      <material
-        name="">
-        <color
-          rgba="0.79216 0.81961 0.93333 1" />
-      </material>
-    </visual>
-    <collision>
-      <origin
-        xyz="0 0 0"
-        rpy="0 0 0" />
-      <geometry>
-        <mesh
-          filename="package://lbr_description/meshes/iiwa7/pole/pole_link5_1.STL" />
-      </geometry>
-    </collision>
-  </link>
-  <joint
-    name="pole_joint4_1"
-    type="fixed">
-    <origin
-      xyz="0.17219 -0.041994 -0.028068"
-      rpy="2.3562 0 -1.5708" />
-    <parent
-      link="pole_link4" />
+        xyz="1.01858932524679E-07 0.0181558532490662 -0.00217161507290353"
+        rpy="0 0 0" />
+      <mass
+        value="0.387118723628718" />
+      <inertia
+        ixx="0.000483645582581851"
+        ixy="8.74673917311267E-10"
+        ixz="-8.11633891736856E-10"
+        iyy="0.00129147787044201"
+        iyz="1.86444604706742E-05"
+        izz="0.000980309144522967" />
+    </inertial>
+    <visual>
+      <origin
+        xyz="0 0 0"
+        rpy="0 0 0" />
+      <geometry>
+        <mesh
+          filename="package://lbr_description/meshes/pole/pole_link5_1.STL" />
+      </geometry>
+      <material
+        name="">
+        <color
+          rgba="0.792156862745098 0.819607843137255 0.933333333333333 1" />
+      </material>
+    </visual>
+    <collision>
+      <origin
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