Commit message: Fix shaking right robot (in gazebo) caused by collisions with pole

File: lbr_description/urdf/right_arm/right_arm.urdf.xacro (robot description, xacro)
@@ -12,9 +12,18 @@
   <joint name="$(arg base_frame)_joint" type="fixed">
       <origin
-          xyz="-0.2193 -0.27 0.281"
-          rpy="-0.7854 0 1.5708" />
+          xyz="-0.2197 -0.268 0.281"
+          rpy="-0.7853981630 0 1.5708" />
       <parent link="$(arg base_frame)" />
       <child link="link_0" />
   </joint>
+  <!--
+  <joint name="$(arg base_frame)_joint" type="fixed">
+      <origin
+          xyz="0 0 0"
+          rpy="-0.7853981630 0 0" />
+      <parent link="$(arg base_frame)" />
+      <child link="link_0" />
+  </joint>
+  -->
   <xacro:iiwa7 robot_name="$(arg robot_name)" port_id="$(arg port_id)" sim="$(arg sim)" />
 </robot>

Commit message: Added collision with 'torso' and table to the right arm

File: lbr_description/urdf/right_arm/right_arm.urdf.xacro (robot description, xacro)
@@ -10,5 +10,5 @@
     <link name="$(arg base_frame)" />
     <!--joint between {base_frame} and link_0-->
-  <joint name="$(arg base_frame)_joint" type="fixed">
+  <joint name="$(arg base_frame)_to_right_arm" type="fixed">
       <origin
           xyz="-0.2197 -0.268 0.281"
@@ -27,3 +27,179 @@
   -->
   <xacro:iiwa7 robot_name="$(arg robot_name)" port_id="$(arg port_id)" sim="$(arg sim)" />
+  <!-- Make sure it doesn't collide with table or pole -->
+  <joint name="$(arg base_frame)_to_table" type="fixed">
+    <parent link="$(arg base_frame)"/>
+    <child link="table"/>
+    <origin xyz="0 0 0" rpy="0 0 0"/>
+  </joint>
+  <link name="table">
+      <collision>
+        <geometry>
+          <box size="1.1 1.1 0.05"/>
+        </geometry>
+      </collision>
+  </link>
+  <joint name="table_to_pole" type="fixed">
+    <parent link="table"/>
+    <child link="base_link"/>
+    <origin xyz="0 -0.35 0.015" rpy="0 0 0"/>
+  </joint>
+ <link
+    name="base_link">
+    <collision>
+      <origin
+        xyz="0 0 0"
+        rpy="0 0 0" />
+      <geometry>
+        <mesh
+          filename="package://lbr_description/meshes/pole/base_link.STL" />
+      </geometry>
+    </collision>
+  </link>
+  <link
+    name="camera_mount">
+    <collision>
+      <origin
+        xyz="0 0 0"
+        rpy="0 0 0" />
+      <geometry>
+        <mesh
+          filename="package://lbr_description/meshes/pole/camera_mount.STL" />
+      </geometry>
+    </collision>
+  </link>
+  <joint
+    name="base_to_camera_mount"
+    type="fixed">
+    <origin
+      xyz="-0.045 0 0.6319"
+      rpy="3.14159265358979 0 -1.5707963267949" />
+    <parent
+      link="base_link" />
+    <child
+      link="camera_mount" />
+    <axis
+      xyz="0 0 0" />
+  </joint>
+  <link
+    name="camera_base">
+    <inertial>
+      <origin
+        xyz="0.00152788225160483 -3.4246869961186E-07 0.0122350480077058"
+        rpy="0 0 0" />
+    </inertial>
+  </link>
+  <joint
+    name="camera_mount_to_camera"
+    type="fixed">
+    <origin
+      xyz="-0.0615 -0.045 -0.0545999999999999"
+      rpy="-3.14159265358979 -0.97738438111683 3.14159265358979" />
+    <parent
+      link="camera_mount" />
+    <child
+      link="camera_base" />
+    <axis
+      xyz="0 0 0" />
+  </joint>
+  <link
+    name="pole_link5_1">
+    <collision>
+      <origin
+        xyz="0 0 0"
+        rpy="0 0 0" />
+      <geometry>
+        <mesh
+          filename="package://lbr_description/meshes/pole/pole_link5_1.STL" />
+      </geometry>
+    </collision>
+  </link>
+  <joint
+    name="base_to_link5_1"
+    type="fixed">
+    <origin
+      xyz="0.212228166945128 0.0800000000000014 0.233931963924182"
+      rpy="-2.35619449019234 0 -1.5707963267949" />
+    <parent
+      link="base_link" />
+    <child
+      link="pole_link5_1" />
+    <axis
+      xyz="0 0 0" />
+  </joint>
+  <link
+    name="pole_link6_1">
+    <collision>
+      <origin
+        xyz="0 0 0"
+        rpy="0 0 0" />
+      <geometry>
+        <mesh
+          filename="package://lbr_description/meshes/pole/pole_link6_1.STL" />
+      </geometry>
+    </collision>
+  </link>
+  <joint
+    name="link5_1_to_link6_1"
+    type="fixed">
+    <origin
+      xyz="0 -0.00999999999999984 0"
+      rpy="-1.5707963267949 3.14159265359 0" />
+    <parent
+      link="pole_link5_1" />
+    <child
+      link="pole_link6_1" />
+    <axis
+      xyz="0 0 0" />
+  </joint>
+  <link
+    name="pole_link5_2">
+    <collision>
+      <origin
+        xyz="0 0 0"
+        rpy="0 0 0" />
+      <geometry>
+        <mesh
+          filename="package://lbr_description/meshes/pole/pole_link5_2.STL" />
+      </geometry>
+    </collision>
+  </link>
+  <joint
+    name="base_to_link5_2"
+    type="fixed">
+    <origin
+      xyz="-0.212192176453971 0.0819943174630784 0.233931963924181"
+      rpy="2.35619449019234 0 1.5707963267949" />
+    <parent
+      link="base_link" />
+    <child
+      link="pole_link5_2" />
+    <axis
+      xyz="0 0 0" />
+  </joint>
+  <link
+    name="pole_link6_2">
+    <collision>
+      <origin
+        xyz="0 0 0"
+        rpy="0 0 0" />
+      <geometry>
+        <mesh
+          filename="package://lbr_description/meshes/pole/pole_link6_2.STL" />
+      </geometry>
+    </collision>
+  </link>
+  <joint
+    name="link5_2_to_link6_2"
+    type="fixed">
+    <origin
+      xyz="0 0 -0.01"
+      rpy="0 0 0" />
+    <parent
+      link="pole_link5_2" />
+    <child
+      link="pole_link6_2" />
+    <axis
+      xyz="0 0 0" />
+  </joint>
 </robot>

Commit message: Update right_arm.urdf.xacro

File: lbr_description/urdf/right_arm/right_arm.urdf.xacro (robot description, xacro)
@@ -88,4 +88,13 @@
         xyz="0.00152788225160483 -3.4246869961186E-07 0.0122350480077058"
         rpy="0 0 0" />
+      <mass
+        value="0.0481481386626754" />
+      <inertia
+        ixx="2.73639159474837E-05"
+        ixy="-4.26051115035423E-07"
+        ixz="7.54720864413178E-09"
+        iyy="3.35044769883872E-06"
+        iyz="2.12843084673675E-09"
+        izz="2.66245899513959E-05" />
     </inertial>
   </link>

Commit message: Fixed URDF for right arm to work with Kinpy

File: lbr_description/urdf/right_arm/right_arm.urdf.xacro (robot description, xacro)
@@ -14,5 +14,5 @@
           xyz="-0.2197 -0.268 0.281"
           rpy="-0.7853981630 0 1.5708" />
-      <parent link="$(arg base_frame)" />
+      <parent link="table" />
       <child link="link_0" />
   </joint>
